Commit message: Create basic urdf visual

File: src/omnibot_description/urdf/omnibot.urdf (robot description, URDF)
Before this commit: robot omnibot, 6 links, 5 joints
Links:
- removed link front_castor_of_wheel
- removed link front_wheel
- added link back_wheel; visual cylinder length=0.026 radius=0.029
- link base_link: mass 1 -> None; geometry visual cylinder length=0.035 radius=0.08
- link left_wheel: mass 1 -> None; geometry visual cylinder length=0.026 radius=0.029
- link right_wheel: mass 1 -> None; geometry visual cylinder length=0.026 radius=0.029
Joints:
- removed joint base_to_castor_socket
- removed joint castor_socket_to_front_wheel
- added joint base_link_to_back_wheel: type continuous, parent base_link, child back_wheel, origin xyz=0.0 -0.08 -0.02 rpy=-1.5707963 0 0, axis 0 0 1
- joint base_foorprint_to_base_link: origin xyz=0 0 0.0512 -> xyz=0 0 0.041
- joint base_link_to_left_wheel: axis 0 0 -1  -> 0 0 1; origin xyz=0.0267 -0.13 -0.02 rpy=-1.57079632679 0  0  -> xyz=-0.069282 0.040 -0.020 rpy=1.5707963 0 1.0471976
- joint base_link_to_right_wheel: origin xyz=0.0267 0.13 -0.02 rpy=1.57079632679 0  0  -> xyz=0.069282 0.040 -0.020 rpy=1.5707963 0 -1.0471976

Commit message: Create xacro

File: src/omnibot_description/urdf/omnibot.urdf (robot description, URDF)
Before this commit: robot omnibot, 5 links, 4 joints
Links:
- removed link back_wheel
- removed link left_wheel
- removed link right_wheel
Joints:
- removed joint base_foorprint_to_base_link
- removed joint base_link_to_back_wheel
- removed joint base_link_to_left_wheel
- removed joint base_link_to_right_wheel
- added joint base_footprint_to_base_link: type fixed, parent base_footprint, child base_link, origin xyz=0 0 0.041
